File: rp2040_stamp_macropad.kicad_pcb (KiCad board)
At the start: 2 copper layers, 100 x 86 mm, 45 parts, among them J1 USB_C_Receptacle_USB2.0, SW1 SW_SPST, SW10 SW_SPST, SW11 SW_SPST, SW12 SW_SPST, SW13 SW_LEFT, SW14 SW_CENTER, SW15 SW_RIGHT, SW2 SW_SPST, SW3 SW_SPST, SW4 SW_SPST, SW5 SW_SPST, SW6 SW_SPST, SW7 SW_SPST, SW8 SW_SPST, SW9 SW_SPST, U1 RP2040_Stamp

Commit message: Rev 2
Parts:
- added J2: Conn_GPIOs, Connector_PinHeader_2.54mm:PinHeader_1x10_P2.54mm_Vertical, B.Cu at (187.5, 124.2)
- added kibuzzard-62DF061F: G***, kibuzzard-62DF061F, F.Cu at (187.4, 122.1)
- added kibuzzard-62DF061F: G***, kibuzzard-62DF061F, B.Cu at (187.4, 121.9)
- added kibuzzard-62DF0636: G***, kibuzzard-62DF0636, F.Cu at (190.0, 122.1)
- added kibuzzard-62DF0636: G***, kibuzzard-62DF0636, B.Cu at (189.9, 121.9)
- added kibuzzard-62DF063C: G***, kibuzzard-62DF063C, F.Cu at (192.5, 122.1)
- added kibuzzard-62DF063C: G***, kibuzzard-62DF063C, B.Cu at (192.5, 122.0)
- added kibuzzard-62DF0641: G***, kibuzzard-62DF0641, F.Cu at (195.0, 122.1)
- added kibuzzard-62DF0641: G***, kibuzzard-62DF0641, B.Cu at (195.0, 122.0)
- added kibuzzard-62DF0644: G***, kibuzzard-62DF0644, F.Cu at (197.6, 122.1)
- added kibuzzard-62DF0644: G***, kibuzzard-62DF0644, B.Cu at (197.6, 121.9)
- added kibuzzard-62DF0648: G***, kibuzzard-62DF0648, F.Cu at (200.1, 122.1)
- added kibuzzard-62DF0648: G***, kibuzzard-62DF0648, B.Cu at (200.1, 121.9)
- added kibuzzard-62DF064B: G***, kibuzzard-62DF064B, F.Cu at (202.7, 122.1)
- added kibuzzard-62DF064B: G***, kibuzzard-62DF064B, B.Cu at (202.6, 122.0)
- added kibuzzard-62DF0650: G***, kibuzzard-62DF0650, F.Cu at (205.2, 121.9)
- added kibuzzard-62DF0650: G***, kibuzzard-62DF0650, B.Cu at (205.2, 121.8)
- added kibuzzard-62DF06D5: G***, kibuzzard-62DF06D5, F.Cu at (207.8, 121.7)
- added kibuzzard-62DF06D5: G***, kibuzzard-62DF06D5, B.Cu at (207.8, 121.6)
- added kibuzzard-62DF06DC: G***, kibuzzard-62DF06DC, F.Cu at (210.3, 121.3)
- added kibuzzard-62DF06DC: G***, kibuzzard-62DF06DC, B.Cu at (210.3, 121.2)
Connections:
- U1 pad 14: unconnected-(U1-Pad14) -> /GPIO13
- U1 pad 15: unconnected-(U1-Pad15) -> /GPIO14
- U1 pad 16: unconnected-(U1-Pad16) -> /GPIO15
- U1 pad 17: unconnected-(U1-Pad17) -> /GPIO16
- U1 pad 18: unconnected-(U1-Pad18) -> /GPIO17
- U1 pad 19: unconnected-(U1-Pad19) -> /GPIO18
- U1 pad 20: unconnected-(U1-Pad20) -> /GPIO19
- U1 pad 21: unconnected-(U1-Pad21) -> /GPIO20
Routing:
- net +3.3V: track 288.8 -> 325.7 mm
- net /GPIO20: track 0.00 -> 14.6 mm
- net /GPIO13: track 0.00 -> 12.8 mm
- net /GPIO14: track 0.00 -> 12.2 mm
- net /GPIO15: track 0.00 -> 11.7 mm
- net /GPIO16: track 0.00 -> 11.2 mm
- net /GPIO17: track 0.00 -> 10.6 mm
- net /GPIO18: track 0.00 -> 10.1 mm
- net /GPIO19: track 0.00 -> 9.56 mm
- net unconnected-(U1-Pad21): track 1.55 -> 0.00 mm
- net unconnected-(U1-Pad20): track 1.55 -> 0.00 mm
- net unconnected-(U1-Pad19): track 1.55 -> 0.00 mm
- net unconnected-(U1-Pad18): track 1.55 -> 0.00 mm
- net unconnected-(U1-Pad17): track 1.55 -> 0.00 mm
- net unconnected-(U1-Pad16): track 1.55 -> 0.00 mm
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