File: rp2040_stamp_macropad.kicad_sch (KiCad schematic)
At the start: 37 parts, among them J1 USB_C_Receptacle_USB2.0, SW1 SW_SPST, SW10 SW_SPST, SW11 SW_SPST, SW12 SW_SPST, SW13 SW_LEFT, SW14 SW_CENTER, SW15 SW_RIGHT, SW2 SW_SPST, SW3 SW_SPST, SW4 SW_SPST, SW5 SW_SPST, SW6 SW_SPST, SW7 SW_SPST, SW8 SW_SPST, SW9 SW_SPST, U1 RP2040_Stamp

Commit message: Rev 2
Parts:
- added J2: (no value), symbol Connector_Generic:Conn_01x10
- C1, C2, C3, C4: value 1uF -> (none); footprint Capacitor_SMD:C_0603_1608Metric -> (none)
- D1, D10, D11, D12, D2, D3, D4, D5, D6, D7, D8, D9: value WS2812B-2020 -> (none); footprint LED_SMD_Extra:WS2812B-2020 -> (none); LCSC (none) -> C965555
- DS1: value OLED-128O064D -> (none); footprint Display:OLED-128O064D -> (none)
- J1: value USB_C_Receptacle_USB2.0 -> (none); footprint Connector_USB:USB_C_Receptacle_HRO_TYPE-C-31-M-12 -> (none); LCSC (none) -> C319148
- R1, R2: value 5.1K -> (none); footprint Resistor_SMD:R_0603_1608Metric -> (none)
- R3: value 390K -> (none); footprint Resistor_SMD:R_0603_1608Metric -> (none)
- SW1, SW10, SW11, SW12, SW2, SW3, SW4, SW5, SW6, SW7, SW8, SW9: value SW_SPST -> (none); footprint Button_Switch_Keyboard:SW_Cherry_MX_1.00u_PCB -> (none)
- SW13: value SW_LEFT -> (none); footprint Button_Switch_SMD:SW_SPST_PTS645 -> (none); LCSC (none) -> C381038
- SW14: value SW_CENTER -> (none); footprint Button_Switch_SMD:SW_SPST_PTS645 -> (none); LCSC (none) -> C381038
- SW15: value SW_RIGHT -> (none); footprint Button_Switch_SMD:SW_SPST_PTS645 -> (none); LCSC (none) -> C381038
- U1: value RP2040_Stamp -> (none); footprint RP2040_Stamp:RP2040_Stamp_FlexyPin -> (none)
Connections:
- net +3.3V: now also J2.9 (Pin_9)
- net GND: now also J2.10 (Pin_10)
- net GPIO13: now reaches U1.14 (GPIO13)
- net GPIO13: now also J2.1 (Pin_1)
- net GPIO14: now reaches U1.15 (GPIO14)
- net GPIO14: now also J2.2 (Pin_2)
- net GPIO15: now reaches U1.16 (GPIO15)
- net GPIO15: now also J2.3 (Pin_3)
- net GPIO16: now reaches U1.17 (GPIO16)
- net GPIO16: now also J2.4 (Pin_4)
- net GPIO17: now reaches U1.18 (GPIO17)
- net GPIO17: now also J2.5 (Pin_5)
- net GPIO18: now reaches U1.19 (GPIO18)
- net GPIO18: now also J2.6 (Pin_6)
- net GPIO19: now reaches U1.20 (GPIO19)
- net GPIO19: now also J2.7 (Pin_7)
- net GPIO20: now reaches U1.21 (GPIO20)
- net GPIO20: now also J2.8 (Pin_8)
- no-connect marks 24 -> 16
